File: power.sch (EAGLE design)
At the start: 20 parts, among them CON1 PINHEAD_2X02-0877590414, CON2 PINHEAD_2X02-0877590414, CON3 PINHEAD_2X02-0877590414, CON5 PINHEAD_2X02-0877590414, CON6 PINHEAD_2X04-SMD-2-MALE, IC1 UCC272-VDFN-HEAVY_PCB, IC2 UCC272-VDFN-HEAVY_PCB, IC3 UCC272-VDFN-HEAVY_PCB

Commit message: Attributes extension
Parts:
- IC1, IC2, IC3: LCSC# (none) -> C47661
Changed lines of the file:
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@@
 </part>
 <part name="GND2" library="supply_symbols" library_urn="urn:adsk.eagle:library:5017758" deviceset="PGND" device="" value="PGND"/>
-<part name="IC1" library="mosfet_drivers" library_urn="urn:adsk.eagle:library:7691028" deviceset="UCC272" device="-VDFN-HEAVY_PCB" package3d_urn="urn:adsk.eagle:package:23775086/3"/>
+<part name="IC1" library="mosfet_drivers" library_urn="urn:adsk.eagle:library:7691028" deviceset="UCC272" device="-VDFN-HEAVY_PCB" package3d_urn="urn:adsk.eagle:package:23775086/3">
+<attribute name="LCSC#" value="C47661"/>
+</part>
 <part name="+P3" library="supply_symbols" library_urn="urn:adsk.eagle:library:13097679" deviceset="15V" device=""/>
 <part name="GND5" library="supply_symbols" library_urn="urn:adsk.eagle:library:5017758" deviceset="PGND" device="" value="PGND"/>
@@
 </part>
 <part name="GND6" library="supply_symbols" library_urn="urn:adsk.eagle:library:5017758" deviceset="PGND" device="" value="PGND"/>
-<part name="IC2" library="mosfet_drivers" library_urn="urn:adsk.eagle:library:7691028" deviceset="UCC272" device="-VDFN-HEAVY_PCB" package3d_urn="urn:adsk.eagle:package:23775086/3"/>
+<part name="IC2" library="mosfet_drivers" library_urn="urn:adsk.eagle:library:7691028" deviceset="UCC272" device="-VDFN-HEAVY_PCB" package3d_urn="urn:adsk.eagle:package:23775086/3">
+<attribute name="LCSC#" value="C47661"/>
+</part>
 <part name="+P4" library="supply_symbols" library_urn="urn:adsk.eagle:library:13097679" deviceset="15V" device=""/>
 <part name="GND1" library="supply_symbols" library_urn="urn:adsk.eagle:library:5017758" deviceset="PGND" device="" value="PGND"/>
@@
 </part>
 <part name="GND3" library="supply_symbols" library_urn="urn:adsk.eagle:library:5017758" deviceset="PGND" device="" value="PGND"/>
-<part name="IC3" library="mosfet_drivers" library_urn="urn:adsk.eagle:library:7691028" deviceset="UCC272" device="-VDFN-HEAVY_PCB" package3d_urn="urn:adsk.eagle:package:23775086/3"/>
+<part name="IC3" library="mosfet_drivers" library_urn="urn:adsk.eagle:library:7691028" deviceset="UCC272" device="-VDFN-HEAVY_PCB" package3d_urn="urn:adsk.eagle:package:23775086/3">
+<attribute name="LCSC#" value="C47661"/>
+</part>
 <part name="+P5" library="supply_symbols" library_urn="urn:adsk.eagle:library:13097679" deviceset="15V" device=""/>
 <part name="GND7" library="supply_symbols" library_urn="urn:adsk.eagle:library:5017758" deviceset="PGND" device="" value="PGND"/>
@@
 <attribute name="NAME" x="90.17" y="164.084" size="2.54" layer="95" font="vector" ratio="15" rot="MR0" align="center"/>
 <attribute name="MANF#" x="90.17" y="140.716" size="1.778" layer="95" font="vector" ratio="15" rot="MR0" align="center"/>
+<attribute name="LCSC#" x="99.06" y="142.24" size="1.27" layer="96" rot="MR0" display="off"/>
 </instance>
 <instance part="+P3" gate="G$1" x="104.14" y="165.1" smashed="yes">
@@
 <attribute name="NAME" x="90.17" y="103.124" size="2.54" layer="95" font="vector" ratio="15" rot="MR0" align="center"/>
 <attribute name="MANF#" x="90.17" y="79.756" size="1.778" layer="95" font="vector" ratio="15" rot="MR0" align="center"/>
+<attribute name="LCSC#" x="99.06" y="81.28" size="1.27" layer="96" rot="MR0" display="off"/>
 </instance>
 <instance part="+P4" gate="G$1" x="104.14" y="104.14" smashed="yes">
@@
 <attribute name="NAME" x="90.17" y="133.604" size="2.54" layer="95" font="vector" ratio="15" rot="MR0" align="center"/>
 <attribute name="MANF#" x="90.17" y="110.236" size="1.778" layer="95" font="vector" ratio="15" rot="MR0" align="center"/>
+<attribute name="LCSC#" x="99.06" y="111.76" size="1.27" layer="96" rot="MR0" display="off"/>
 </instance>
 <instance part="+P5" gate="G$1" x="104.14" y="134.62" smashed="yes">
