File: src/logic.brd (EAGLE design)
At the start: 37.8 x 80 mm, 89 parts, among them CON11 PINHEAD_1X03-2, CON12 PINHEAD_1X03-2, CON2 PINHEAD_2X02-PTH-2-MALE, CON3 PINHEAD_2X04-PLS-2, CON4 CON-3P-TABS, CON5 PINHEAD_2X02-PTH-2-MALE, CON6 PINHEAD_2X02-PTH-2-MALE, CON7 PINHEAD_2X02-PTH-2-MALE, IC1 STM32F105RCT6, IC10 LM75-TSSOP8, IC11 LM75-TSSOP8, IC2 CAT24C02, IC3 AP2127-3.3, IC4 LM75-TSSOP8, IC6 ZXCT1051, IC7 ST3232, IC8 LM75-TSSOP8, X1 16MHz

Commit message: initial import
Parts:
- removed C10: 0.1µF, rc:C0402
- removed C17, C18, C19, C20, C21, C23: 100µF, rc:RADIAL_SIDE_12.5X22
- removed C28: 1µF, C_digikey:C0603
- removed CON2, CON5: PINHEAD_2X02-PTH-2-MALE, pinhead:2X02-PTH-2
- removed CON4: CON-3P-TABS, Connectors:JST_GH-3P-RA
- removed HV_DC-DC:C1: 2.2uF, rc:C1210
- removed HV_DC-DC:C2: 0.47uF, rc:C0805
- removed HV_DC-DC:C3: 0.01uF, rc:C0603
- removed HV_DC-DC:C4: 10uF, rc:C1206
- removed HV_DC-DC:C5: 1uf, rc:C0603
- removed HV_DC-DC:CAC: 0.1uF, rc:C0402
- removed HV_DC-DC:CR: 3300pF, rc:C0402
- removed HV_DC-DC:D1: PMEG3005, Diodes:SOD523
- removed HV_DC-DC:IC1: LM5017, dc-dc:SOIC8-POWERPAD
- removed HV_DC-DC:L3: 120µH, power_inductors:HPC8040NF
- removed HV_DC-DC:R3: 127K, rc:R0805
- removed HV_DC-DC:R4: 14K, rc:R0805
- removed HV_DC-DC:RFB1: 1K, rc:R0402
- removed HV_DC-DC:RFB2: 3K, rc:R0402
- removed HV_DC-DC:RON: 110K, rc:R0805
- removed HV_DC-DC:RRIP: 110K, rc:R0402
- removed IC2: CAT24C02, misc:SOT23-5L
- removed IC6: ZXCT1051, misc:SOT23-5L
- removed LV_DC-DC:2: 10K, rc:R0402
- removed LV_DC-DC:C1, LV_DC-DC:C2, LV_DC-DC:C3: 10uF, rc:C0805
- removed LV_DC-DC:IC1: TPS62160QDSGRQ1, dc-dc:WFDFN-8
- removed LV_DC-DC:L1: 2.2µH, power_inductors:NR3015
- removed LV_DC-DC:R1: 51K, rc:R0402
- removed R12: 3K9, R_digikey:R0402
- added 202: 10K, rc:R0402
- added C101: 2.2uF, rc:C1210
- added C102: 0.47uF, rc:C0805
- added C103: 0.01uF, rc:C0603
- added C104: 10uF, rc:C1206
- added C105: 1uf, rc:C0603
- added C14: 0.1µF, rc:C0402
- added C201, C202, C203: 10uF, rc:C0805
- added CAC100: 0.1uF, rc:C0402
- added CON1: CON-4P-TABS-JST_GH-RA, Connectors:JST_GH-4P-RA
- added CR100: 3300pF, rc:C0402
- added D101: PMEG3005, Diodes:SOD523
- added IC101: LM5017, dc-dc:SOIC8-POWERPAD
- added IC201: TPS62160QDSGRQ1, dc-dc:WFDFN-8
- added IC5: INA180A1, misc:SOT23-5
- added L103: 120µH, power_inductors:HPC8040NF
- added L201: 2.2µH, power_inductors:NR3015
- added R103: 127K, rc:R0805
- added R104: 14K, rc:R0805
- added R201: 51K, rc:R0402
- added RFB101: 1K, rc:R0402
- added RFB102: 3K, rc:R0402
- added RON100: 110K, rc:R0805
- added RRIP100: 110K, rc:R0402
- moved IC4 165.5 mm to (-13.2, 67.5), flipped to the bottom, turned to 270 degrees
- moved C12 162.8 mm to (43.5, 27.4)
- moved IC7 32.5 mm to (17.4, 80.4)
- moved C2 25.4 mm to (-37.5, 61.4)
- moved C32 25.4 mm to (-37.5, 59.8)
- moved C33 25.4 mm to (-37.5, 58.2)
- moved C34 25.4 mm to (-37.5, 56.6)
- moved C37 25.4 mm to (-37.5, 55.0)
- moved C1 25.1 mm to (-38.5, 66.7)
- moved C31 23.4 mm to (-36.9, 67.3)
- moved IC1 21.6 mm to (9.10, 46.2)
- moved X1 17.1 mm to (5.70, 53.9)
- moved R4 16.0 mm to (10.9, 55.1)
- moved R2 14.9 mm to (25.2, 60.0)
- moved R3 14.9 mm to (25.2, 58.0)
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Connections:
- removed net BLABLA: IC6.3, R12.1
- removed net HV_DC-DC:N$10: HV_DC-DC:C5.2, HV_DC-DC:D1.C, HV_DC-DC:IC1.6
- removed net HV_DC-DC:N$11: HV_DC-DC:IC1.4, HV_DC-DC:RON.2
- removed net HV_DC-DC:N$12: HV_DC-DC:C3.1, HV_DC-DC:IC1.7
- removed net HV_DC-DC:N$14: HV_DC-DC:CAC.1, HV_DC-DC:IC1.5, HV_DC-DC:RFB1.2, HV_DC-DC:RFB2.1
- removed net HV_DC-DC:N$17: HV_DC-DC:IC1.3, HV_DC-DC:R3.1, HV_DC-DC:R4.2
- removed net HV_DC-DC:N$2: HV_DC-DC:C3.2, HV_DC-DC:IC1.8, HV_DC-DC:L3.1, HV_DC-DC:RRIP.2
- removed net HV_DC-DC:N$3: HV_DC-DC:CAC.2, HV_DC-DC:CR.2, HV_DC-DC:RRIP.1
- removed net N$1: IC6.5
- removed net N$2: IC6.4
- removed net VBAT: C17.+, C18.+, C19.+, C20.+, C21.+, C23.+
- new net CS+: CON3.7
- new net CS-: CON3.5
- new net HV_DC-DC(LM5017):N$10: C105.2, D101.C, IC101.6
- new net HV_DC-DC(LM5017):N$11: IC101.4, RON100.2
- new net HV_DC-DC(LM5017):N$12: C103.1, IC101.7
- new net HV_DC-DC(LM5017):N$14: CAC100.1, IC101.5, RFB101.2, RFB102.1
- new net HV_DC-DC(LM5017):N$17: IC101.3, R103.1, R104.2
- new net HV_DC-DC(LM5017):N$2: C103.2, IC101.8, L103.1, RRIP100.2
- new net HV_DC-DC(LM5017):N$3: CAC100.2, CR100.2, RRIP100.1
- new net N$5: IC5.3
- new net N$8: IC5.4
- new net RCPWM: CON1.1
- new net VBAT-: CON3.3
- net FET_A_H: now also CON6.2
- net FET_A_L: now also CON6.4
- net FET_C_H: now also CON3.2, CON7.2
- net FET_C_L: now also CON3.4, CON7.4
- net GND: now also 202.1, 202.2, C101.1, C102.1, C104.P$1, C105.1, C14.2, C201.1, C202.1, C203.1, CON1.4, CON1.M$0, CON1.M$1, IC101.1, IC101.P$1, IC201.1, IC201.4, IC201.5, IC201.EP, IC5.2, R104.1, R201.1, RFB101.1; no longer C10.2, C17.-, C18.-, C19.-, C20.-, C21.-, C23.-, C28.P$1, CON4.3, CON4.M$0, CON4.M$1, HV_DC-DC:C1.1, HV_DC-DC:C2.1, HV_DC-DC:C4.P$1, HV_DC-DC:C5.1, HV_DC-DC:IC1.1, HV_DC-DC:IC1.P$1, HV_DC-DC:R4.1, HV_DC-DC:RFB1.1, IC2.2, IC6.2, LV_DC-DC:2.1, LV_DC-DC:2.2, LV_DC-DC:C1.1, LV_DC-DC:C2.1, LV_DC-DC:C3.1, LV_DC-DC:IC1.1, LV_DC-DC:IC1.4, LV_DC-DC:IC1.5, LV_DC-DC:IC1.EP, LV_DC-DC:R1.1
- net I2C_SCL: no longer IC2.1
- net I2C_SDA: no longer IC2.3
- net LV_DC-DC:N$1: now also IC201.7, L201.1; no longer LV_DC-DC:IC1.7, LV_DC-DC:L1.1
- net N$29: now also CON1.3; no longer CON4.2
- net N$30: now also CON1.2; no longer CON4.1
- net PHASE_A: now also CON6.3
- net PHASE_B: now also CON7.3
- net PHASE_C: now also CON3.8
- net SENSE_CURRENT: now also IC5.1; no longer C28.P$2, R12.2
- net VDC: now also C101.2, C102.2, CON3.1, IC101.2, R103.2, RON100.1; no longer HV_DC-DC:C1.2, HV_DC-DC:C2.2, HV_DC-DC:IC1.2, HV_DC-DC:R3.2, HV_DC-DC:RON.1
- net VDD_12V: now also C104.P$2, C201.2, CON3.6, CON6.1, CON7.1, CR100.1, D101.A, IC201.2, IC201.3, L103.2, RFB102.2; no longer HV_DC-DC:C4.P$2, HV_DC-DC:CR.1, HV_DC-DC:D1.A, HV_DC-DC:L3.2, HV_DC-DC:RFB2.2, LV_DC-DC:C1.2, LV_DC-DC:IC1.2, LV_DC-DC:IC1.3
- net VDD_3V3: now also C14.1, IC5.5; no longer C10.1, IC2.4, IC6.1
- net VDD_5V: now also C202.2, C203.2, IC201.6, L201.2, R201.2; no longer LV_DC-DC:C2.2, LV_DC-DC:C3.2, LV_DC-DC:IC1.6, LV_DC-DC:L1.2, LV_DC-DC:R1.2
Other:
- board size 37.8 x 80 mm -> 36 x 80 mm

Commit message: Connectors update
Connections:
- removed net N$5: IC5.3
- removed net N$8: IC5.4
- net CS+: now also IC5.3
- net CS-: now also IC5.4
Changed lines of the file:
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@@
 <contactref element="CON1" pad="1"/>
-</signal>
-<signal name="N$5">
-<contactref element="IC5" pad="3"/>
-</signal>
-<signal name="N$8">
-<contactref element="IC5" pad="4"/>
 </signal>
 <signal name="CS+">
 <contactref element="CON3" pad="7"/>
+<contactref element="IC5" pad="3"/>
+<wire x1="-10.5" y1="72.35" x2="-6.15" y2="72.4" width="0" layer="19" extent="1-1"/>
 </signal>
 <signal name="CS-">
 <contactref element="CON3" pad="5"/>
+<contactref element="IC5" pad="4"/>
+<wire x1="-13.1" y1="72.35" x2="-6.15" y2="74.4" width="0" layer="19" extent="1-1"/>
 </signal>
 <signal name="VBAT-">

Commit message: Components placement
Parts:
- removed 202: 10K, rc:R0402
- added C10: 0.1µF, C_digikey:C0402
- added IC2: CAT24C02, misc:SOT23-5L
- added R1: 000, rc:R0805
- added R202: 10K, rc:R0402
- D1, D2, D4: value BAS16L -> BAT54KFILM; device Diodes:SOD882 -> Diodes:SOD523
- R104: device rc:R0805 -> rc:R0402
- X1: device crystal:OSCILLATOR-2.0X1.6-4P -> crystal:OSCILLATOR-3.2X2.5-4P
- moved CAC100 57.3 mm to (-11.9, 37.3), turned to 180 degrees
- moved RRIP100 56.3 mm to (-11.9, 34.9)
- moved CR100 56.3 mm to (-11.9, 36.1), turned to 180 degrees
- moved C25 49.5 mm to (-2.90, 65.4), turned to 270 degrees
- moved RON100 48.9 mm to (-12.9, 41.6)
- moved R11 46.8 mm to (-4.00, 65.4), turned to 270 degrees
- moved C101 45.4 mm to (-10.2, 49.1), turned to 0 degrees
- moved C102 43.8 mm to (-7.20, 46.4), turned to 180 degrees
- moved R103 43.7 mm to (-10.8, 46.4), turned to 180 degrees
- moved R10 43.4 mm to (-5.50, 64.7), turned to 270 degrees
- moved C31 42.3 mm to (5.12, 72.8), turned to 135 degrees
- moved C103 40.5 mm to (-6.60, 36.8)
- moved C3 40.4 mm to (0.52, 67.9), turned to 315 degrees
- moved D101 40.2 mm to (-4.70, 37.3), turned to 270 degrees
- moved C1 39.9 mm to (1.30, 68.7), turned to 315 degrees
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Connections:
- new net LV_DC-DC:FB: IC201.5, R201.1, R202.2
- net GND: now also C10.2, IC2.2, R202.1; no longer 202.1, 202.2, IC201.5, R201.1
- net I2C_SCL: now also IC2.1
- net I2C_SDA: now also IC2.3
- net VDD_3V3: now also C10.1, IC2.4, R1.2
- net VDD_5V: now also R1.1
Routing:
- net HV_DC-DC(LM5017):N$2: track 0.00 -> 8.44 mm
- net I2C_SCL: track 0.00 -> 7.10 mm
- net I2C_SDA: track 0.00 -> 5.29 mm
- net VDD_3V3: track 0.00 -> 5.14 mm
- net HV_DC-DC(LM5017):N$14: track 0.00 -> 4.20 mm
- net BOOT0: track 0.00 -> 2.45 mm
- net HV_DC-DC(LM5017):N$3: track 0.00 -> 2.40 mm
- net HV_DC-DC(LM5017):N$12: track 0.00 -> 1.94 mm
- net HV_DC-DC(LM5017):N$10: track 0.00 -> 1.94 mm

Commit message: Update logic.brd
Parts:
- moved IC8 5.15 mm to (-5.00, 19.0)
Other:
- board size 36 x 80 mm -> 36 x 63 mm
Changed lines of the file:
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@@
 <layer number="14" name="Route14" color="22" fill="1" visible="no" active="no"/>
 <layer number="15" name="Route15" color="23" fill="1" visible="no" active="yes"/>
-<layer number="16" name="Bottom" color="1" fill="1" visible="no" active="yes"/>
+<layer number="16" name="Bottom" color="1" fill="1" visible="yes" active="yes"/>
 <layer number="17" name="Pads" color="2" fill="1" visible="yes" active="yes"/>
 <layer number="18" name="Vias" color="2" fill="1" visible="yes" active="yes"/>
@@
 <layer number="20" name="Dimension" color="24" fill="1" visible="yes" active="yes"/>
 <layer number="21" name="tPlace" color="7" fill="1" visible="yes" active="yes"/>
-<layer number="22" name="bPlace" color="7" fill="1" visible="no" active="yes"/>
+<layer number="22" name="bPlace" color="7" fill="1" visible="yes" active="yes"/>
 <layer number="23" name="tOrigins" color="15" fill="1" visible="yes" active="yes"/>
-<layer number="24" name="bOrigins" color="15" fill="1" visible="no" active="yes"/>
+<layer number="24" name="bOrigins" color="15" fill="1" visible="yes" active="yes"/>
 <layer number="25" name="tNames" color="7" fill="1" visible="yes" active="yes"/>
-<layer number="26" name="bNames" color="7" fill="1" visible="no" active="yes"/>
+<layer number="26" name="bNames" color="7" fill="1" visible="yes" active="yes"/>
 <layer number="27" name="tValues" color="7" fill="1" visible="no" active="yes"/>
 <layer number="28" name="bValues" color="7" fill="1" visible="no" active="yes"/>
@@
 <layer number="50" name="dxf" color="7" fill="1" visible="no" active="no"/>
 <layer number="51" name="tDocu" color="7" fill="1" visible="yes" active="yes"/>
-<layer number="52" name="bDocu" color="7" fill="1" visible="no" active="yes"/>
+<layer number="52" name="bDocu" color="7" fill="1" visible="yes" active="yes"/>
 <layer number="53" name="tGND_GNDA" color="7" fill="9" visible="no" active="no"/>
 <layer number="54" name="bGND_GNDA" color="1" fill="9" visible="no" active="no"/>
@@
 </layers>
 <board>
-<fusionsync huburn="a.cGVyc29uYWw6dWUyYWE4ZDY4" projecturn="a.cGVyc29uYWw6dWUyYWE4ZDY4IzIwMjAwOTI1MzM2NDYxMjgx" f3durn="urn:adsk.wipprod:dm.lineage:ZtDsZR-uQpiuHdusn4WlVw" pcbguid="" lastpulledtime="" lastsyncedchangeguid="" latestrevisionid="75ea08a6-7ba3-4ca6-b257-1ddbba0a3e16" lastsyncedrevisionid="75ea08a6-7ba3-4ca6-b257-1ddbba0a3e16" lastboardhashguid="03b4536f-98e4-5604-86a3-fbb45b2e6015" lastpushedtime="2020-10-28T12:53:15Z" linktopcb3d="true"/>
+<fusionsync huburn="a.cGVyc29uYWw6dWUyYWE4ZDY4" projecturn="a.cGVyc29uYWw6dWUyYWE4ZDY4IzIwMjAwOTI1MzM2NDYxMjgx" f3durn="urn:adsk.wipprod:dm.lineage:ZtDsZR-uQpiuHdusn4WlVw" pcbguid="" lastpulledtime="" lastsyncedchangeguid="" latestrevisionid="98bb935b-9aa4-4de4-9b09-5cdbe39f2b6c" lastsyncedrevisionid="98bb935b-9aa4-4de4-9b09-5cdbe39f2b6c" lastboardhashguid="7631717c-786e-be49-bb54-417e5e29b1e3" lastpushedtime="2020-10-29T11:12:54Z" linktopcb3d="true"/>
 <plain>
 <wire x1="0" y1="0" x2="0" y2="80" width="0.01" layer="47" style="shortdash" locked="yes"/>
@@
 <wire x1="8.5" y1="79" x2="8.5" y2="76" width="0.01" layer="20" locked="yes"/>
 <wire x1="8.5" y1="76" x2="10.5" y2="74" width="0.01" layer="20" curve="90" locked="yes"/>
-<wire x1="-17" y1="0" x2="17" y2="0" width="0.01" layer="20" locked="yes"/>
-<wire x1="17" y1="0" x2="18" y2="1" width="0.01" layer="20" curve="90" locked="yes"/>
-<wire x1="18" y1="1" x2="18" y2="55" width="0.01" layer="20" locked="yes"/>
+<wire x1="-17" y1="22" x2="-10" y2="22" width="0.01" layer="20"/>
+<wire x1="-10" y1="22" x2="-9" y2="21" width="0.01" layer="20" curve="-90"/>
+<wire x1="-9" y1="21" x2="-9" y2="18" width="0.01" layer="20"/>
+<wire x1="-9" y1="18" x2="-8" y2="17" width="0.01" layer="20" curve="90"/>
+<wire x1="-8" y1="17" x2="-2" y2="17" width="0.01" layer="20"/>
+<wire x1="-2" y1="17" x2="-1" y2="18" width="0.01" layer="20" curve="90"/>
+<wire x1="-1" y1="18" x2="-1" y2="21" width="0.01" layer="20"/>
+<wire x1="-1" y1="21" x2="0" y2="22" width="0.01" layer="20" curve="-90"/>
+<wire x1="0" y1="22" x2="17" y2="22" width="0.01" layer="20"/>
+<wire x1="17" y1="22" x2="18" y2="23" width="0.01" layer="20" curve="90"/>
+<wire x1="18" y1="23" x2="18" y2="55" width="0.01" layer="20"/>
 <wire x1="18" y1="55" x2="17" y2="56" width="0.01" layer="20" curve="90" locked="yes"/>
 <wire x1="17" y1="56" x2="14.7" y2="56" width="0.01" layer="20" locked="yes"/>
@@
 <wire x1="-14.7" y1="56" x2="-17" y2="56" width="0.01" layer="20" locked="yes"/>
 <wire x1="-17" y1="56" x2="-18" y2="55" width="0.01" layer="20" curve="90" locked="yes"/>
-<wire x1="-18" y1="55" x2="-18" y2="1" width="0.01" layer="20" locked="yes"/>
-<wire x1="-18" y1="1" x2="-17" y2="0" width="0.01" layer="20" curve="90" locked="yes"/>
+<wire x1="-18" y1="55" x2="-18" y2="23" width="0.01" layer="20"/>
+<wire x1="-18" y1="23" x2="-17" y2="22" width="0.01" layer="20" curve="90"/>
 <wire x1="-10.5" y1="74" x2="-8.5" y2="76" width="0.01" layer="20" curve="90" locked="yes"/>
 <rectangle x1="-2.5" y1="62" x2="2.5" y2="70" layer="49"/>
 <rectangle x1="-2.5" y1="36" x2="2.5" y2="44" layer="49"/>
 <rectangle x1="-2.5" y1="10" x2="2.5" y2="18" layer="49"/>
-<wire x1="-2.5" y1="4" x2="-2.5" y2="7" width="0.01" layer="20" locked="yes"/>
-<wire x1="-2.5" y1="7" x2="-1.5" y2="8" width="0.01" layer="20" curve="-90" locked="yes"/>
-<wire x1="-1.5" y1="8" x2="1.5" y2="8" width="0.01" layer="20" locked="yes"/>
-<wire x1="1.5" y1="8" x2="2.5" y2="7" width="0.01" layer="20" curve="-90" locked="yes"/>
-<wire x1="2.5" y1="7" x2="2.5" y2="4" width="0.01" layer="20" locked="yes"/>
-<wire x1="2.5" y1="4" x2="1.5" y2="3" width="0.01" layer="20" curve="-90" locked="yes"/>
-<wire x1="1.5" y1="3" x2="-1.5" y2="3" width="0.01" layer="20" locked="yes"/>
-<wire x1="-1.5" y1="3" x2="-2.5" y2="4" width="0.01" layer="20" curve="-90" locked="yes"/>
 <wire x1="2.5" y1="33" x2="2.5" y2="30" width="0.01" layer="20" locked="yes"/>
 <wire x1="2.5" y1="30" x2="1.5" y2="29" width="0.01" layer="20" curve="-90" locked="yes"/>
@@
 <attribute name="NAME" x="-5.15" y="80" locked="yes" size="1" layer="25" font="vector" ratio="15" align="center"/>
 </element>
-<element name="IC8" library="misc" library_urn="urn:adsk.eagle:library:5347860" package="TSSOP8" package3d_urn="urn:adsk.eagle:package:7691413/6" value="LM75-TSSOP8" x="0" y="17.75" smashed="yes" rot="MR0">
-<attribute name="DIGIKEY#" value="568-4768-1-ND" x="0" y="17.75" size="1.778" layer="28" rot="MR0" display="off"/>
-<attribute name="LCSC#" value="C33099" x="0" y="17.75" size="1.778" layer="28" rot="MR0" display="off"/>
-<attribute name="MANF" value="NXP Semiconductors" x="0" y="17.75" size="1.778" layer="28" rot="MR0" display="off"/>
-<attribute name="MANF#" value="LM75BDP,118" x="0" y="17.75" size="1.778" layer="28" rot="MR0" display="off"/>
-<attribute name="NAME" x="0" y="17.75" size="1.27" layer="26" font="vector" ratio="15" rot="MR0" align="center"/>
+<element name="IC8" library="misc" library_urn="urn:adsk.eagle:library:5347860" package="TSSOP8" package3d_urn="urn:adsk.eagle:package:7691413/6" value="LM75-TSSOP8" x="-5" y="19" smashed="yes" rot="MR0">
+<attribute name="DIGIKEY#" value="568-4768-1-ND" x="-5" y="19" size="1.778" layer="28" rot="MR0" display="off"/>
+<attribute name="LCSC#" value="C33099" x="-5" y="19" size="1.778" layer="28" rot="MR0" display="off"/>
+<attribute name="MANF" value="NXP Semiconductors" x="-5" y="19" size="1.778" layer="28" rot="MR0" display="off"/>
+<attribute name="MANF#" value="LM75BDP,118" x="-5" y="19" size="1.778" layer="28" rot="MR0" display="off"/>
+<attribute name="NAME" x="-5" y="19" size="1.27" layer="26" font="vector" ratio="15" rot="MR0" align="center"/>
 </element>
 <element name="IC10" library="misc" library_urn="urn:adsk.eagle:library:5347860" package="TSSOP8" package3d_urn="urn:adsk.eagle:package:7691413/6" value="LM75-TSSOP8" x="0" y="42.25" smashed="yes" rot="MR0">
@@
 <wire x1="7.5" y1="30" x2="7.5" y2="32" width="0" layer="19" extent="1-1"/>
 <wire x1="7.5" y1="28" x2="7.5" y2="30" width="0" layer="19" extent="1-1"/>
-<wire x1="2.925" y1="16.775" x2="7.5" y2="28" width="0" layer="19" extent="1-16"/>
-<wire x1="-2.925" y1="16.775" x2="2.925" y2="16.775" width="0" layer="19" extent="16-16"/>
-<wire x1="-2.925" y1="17.425" x2="-2.925" y2="16.775" width="0" layer="19" extent="16-16"/>
-<wire x1="-2.925" y1="18.075" x2="-2.925" y2="17.425" width="0" layer="19" extent="16-16"/>
+<wire x1="-2.075" y1="18.025" x2="7.5" y2="28" width="0" layer="19" extent="1-16"/>
+<wire x1="-7.925" y1="18.025" x2="-2.075" y2="18.025" width="0" layer="19" extent="16-16"/>
+<wire x1="-7.925" y1="18.675" x2="-7.925" y2="18.025" width="0" layer="19" extent="16-16"/>
+<wire x1="-7.925" y1="19.325" x2="-7.925" y2="18.675" width="0" layer="19" extent="16-16"/>
 </signal>
 <signal name="SENSE_B">
@@
 <wire x1="2.925" y1="42.575" x2="2.825" y2="53.675" width="0" layer="19" extent="16-16"/>
 <wire x1="-13.525" y1="70.425" x2="2.825" y2="53.675" width="0" layer="19" extent="16-16"/>
-<wire x1="2.925" y1="18.075" x2="2.925" y2="42.575" width="0" layer="19" extent="16-16"/>
+<wire x1="-2.075" y1="19.325" x2="2.925" y2="42.575" width="0" layer="19" extent="16-16"/>
 </signal>
 <signal name="I2C_SDA">
@@
 <wire x1="2.925" y1="43.225" x2="2.825" y2="54.325" width="0" layer="19" extent="16-16"/>
 <wire x1="-14.175" y1="70.425" x2="2.825" y2="54.325" width="0" layer="19" extent="16-16"/>
-<wire x1="2.925" y1="18.725" x2="2.925" y2="43.225" width="0" layer="19" extent="16-16"/>
+<wire x1="-2.075" y1="19.975" x2="2.925" y2="43.225" width="0" layer="19" extent="16-16"/>
 </signal>
 <signal name="USART1_TX">
@@
 <wire x1="6.5" y1="30" x2="6.5" y2="32" width="0" layer="19" extent="1-1"/>
 <wire x1="6.5" y1="28" x2="6.5" y2="30" width="0" layer="19" extent="1-1"/>
-<wire x1="-2.925" y1="18.725" x2="6.5" y2="28" width="0" layer="19" extent="1-16"/>
+<wire x1="-7.925" y1="19.975" x2="6.5" y2="28" width="0" layer="19" extent="1-16"/>
 </signal>
 <signal name="BOOT0">

Commit message: outline update
Parts:
- moved C12 46.5 mm to (-15.0, 69.0), turned to 90 degrees
- moved C29 29.6 mm to (-11.0, 55.5), turned to 90 degrees
- moved C13 17.3 mm to (-5.50, 18.0), turned to 90 degrees
- moved C11 9.22 mm to (0.00, 40.0), flipped to the bottom
- moved IC11 9.10 mm to (-8.90, 55.6), turned to 180 degrees
- moved CAC100 1.50 mm to (-11.9, 38.8)
- moved CR100 1.50 mm to (-11.9, 37.6)
- moved RFB101 1.50 mm to (-11.9, 41.2)
- moved RFB102 1.50 mm to (-11.9, 40.0)
- moved RON100 1.50 mm to (-12.9, 43.1)
- moved RRIP100 1.50 mm to (-11.9, 36.4)
- moved D2 1.12 mm to (-3.80, 55.4)
- moved IC8 0.71 mm to (-5.50, 18.5), turned to 270 degrees
- moved C101 0.50 mm to (-10.2, 49.6)
- moved C102 0.50 mm to (-7.20, 46.9)
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Other:
- board size 36 x 63 mm -> 36 x 65.5 mm

Commit message: Updates here and there
Parts:
- removed LED1: LTST-C19HE1WT, misc:0606
- added C15: 0.1µF, rc:C0402
- added LED2: LED_RGB-2020, rc:LED2020
- added R5: (no value), rc:R0805
- added R6: (no value), rc:R0402
- moved C11 13.1 mm to (13.1, 39.9), flipped to the top
- moved D101 9.96 mm to (-3.20, 47.6), turned to 180 degrees
- moved C104 8.24 mm to (5.80, 41.3), turned to 270 degrees
- moved C22 5.79 mm to (-1.57, 63.4), turned to 135 degrees
- moved R9 5.77 mm to (-0.79, 64.2), turned to 135 degrees
- moved C27 4.82 mm to (16.2, 42.9), turned to 90 degrees
- moved IC10 4.70 mm to (4.70, 42.4)
- moved C203 4.17 mm to (10.8, 47.5), turned to 270 degrees
- moved C26 4.01 mm to (12.8, 45.0)
- moved IC11 3.83 mm to (-11.8, 53.2)
- moved R25 3.52 mm to (9.65, 55.1), turned to 90 degrees
- moved D2 3.51 mm to (-4.10, 58.9), turned to 180 degrees
- moved R1 3.48 mm to (15.5, 46.7)
- moved D4 3.44 mm to (-1.42, 66.4), turned to 135 degrees
- moved C202 3.37 mm to (12.8, 47.5)
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Connections:
- removed net USART1_RX/PWM: IC1.14, IC1.59, IC7.12
- removed net VBAT-: CON3.3
- new net RC_PWM: IC1.14
- new net USART1_RX: IC1.59, IC7.12
- net FET_A_H: now also CON3.2; no longer CON6.2
- net FET_A_L: now also CON3.4; no longer CON6.4
- net FET_B_H: now also CON7.2
- net FET_B_L: now also CON7.4
- net FET_C_H: now also CON6.2; no longer CON3.2, CON7.2
- net FET_C_L: now also CON6.4; no longer CON3.4, CON7.4
- net GND: now also C15.1, CON3.3, R6.1
- net N$26: now also LED2.G; no longer LED1.G
- net N$6: now also LED2.B; no longer LED1.B
- net N$7: now also LED2.R; no longer LED1.R
- net PHASE_A: now also CON3.8, R10.1; no longer CON6.3, R7.1
- net PHASE_C: now also CON6.3, R7.1; no longer CON3.8, R10.1
- net SENSE_A: now also C25.2, D4.A, R10.2, R11.2; no longer C30.2, D2.A, R15.2, R7.2
- net SENSE_C: now also C30.2, D2.A, R15.2, R7.2; no longer C25.2, D4.A, R10.2, R11.2
- net SENSE_VIN: now also C15.2, R5.1, R6.2
- net VDC: now also R5.2
- net VDD_3V3: now also LED2.+; no longer LED1.+
Routing:
- net VDD_12V: track 0.00 -> 54.3 mm
- net FET_C_H: track 0.00 -> 45.6 mm, vias 0 -> 1
- net VDD_3V3: track 5.14 -> 49.1 mm, vias 0 -> 8
- net FET_C_L: track 0.00 -> 43.5 mm, vias 0 -> 1
- net N$7: track 0.00 -> 30.8 mm, vias 0 -> 2
- net N$26: track 0.00 -> 28.6 mm, vias 0 -> 2
- net FET_A_H: track 0.00 -> 25.4 mm, vias 0 -> 1
- net N$6: track 0.00 -> 25.1 mm, vias 0 -> 2
- net FET_B_H: track 0.00 -> 24.6 mm, vias 0 -> 2
- net USART1_TX: track 0.00 -> 23.5 mm, vias 0 -> 2
- net USART1_RX: track 0.00 -> 23.5 mm, vias 0 -> 2
- net FET_A_L: track 0.00 -> 22.5 mm, vias 0 -> 1
- net VDC: track 0.00 -> 22.1 mm
- net N$30: track 0.00 -> 18.7 mm
- net GND: track 0.00 -> 18.3 mm, vias 0 -> 9
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- added copper zone on layer 1, net GND
- added copper zone on layer 16, net GND
- added copper zone on layer 1, net HV_DC-DC(LM5017):N$2
- added copper zone on layer 1, net LV_DC-DC:N$1
- added copper zone on layer 1, net VDD_12V
- added copper zone on layer 1, net VDD_5V
Other:
- outline, holes or cut-outs redrawn
