File: src/logic.brd (EAGLE design)
At the start: 36 x 65.5 mm, 84 parts, among them CON1 CON-4P-TABS-JST_GH-RA, CON11 PINHEAD_1X03-2, CON12 PINHEAD_1X03-2, CON3 PINHEAD_2X04-PLS-2, CON6 PINHEAD_2X02-PTH-2-MALE, CON7 PINHEAD_2X02-PTH-2-MALE, IC1 STM32F105RCT6, IC10 LM75-TSSOP8, IC101 LM5017, IC11 LM75-TSSOP8, IC2 CAT24C02, IC201 TPS62160QDSGRQ1, IC3 AP2127-3.3, IC4 LM75-TSSOP8, IC5 INA180A1, IC7 ST3232, IC8 LM75-TSSOP8, X1 16MHz

Commit message: routing upodates
Parts:
- added CON2: PINHEAD_1X04-2.54, pinhead:1X04-PTH-2.54
- moved C12 6.02 mm to (-19.9, 65.5)
- moved C202 5.22 mm to (8.20, 50.0), turned to 0 degrees
- moved R1 3.70 mm to (11.8, 46.6)
- moved IC11 2.91 mm to (-12.8, 50.5), turned to 90 degrees
- moved C203 2.63 mm to (8.20, 48.1), turned to 0 degrees
- moved IC4 1.64 mm to (-11.9, 66.5)
- moved C5 1.60 mm to (9.00, 72.0), turned to 180 degrees
- moved D1 0.45 mm to (-4.30, 63.6)
- moved R6 0.36 mm to (-5.88, 61.4)
- moved C15 0.36 mm to (-6.66, 62.2)
- moved R4 0.14 mm to (13.5, 68.9)
- moved C37 0.10 mm to (-9.70, 66.8), turned to 180 degrees
Connections:
- net GND: now also CON2.3
- net SWCLK: now also CON2.1
- net SWDIO: now also CON2.2
- net VDD_3V3: now also CON2.4
Routing:
- net VDD_3V3: track 49.1 -> 120.5 mm, vias 8 -> 15
- net VDD_12V: track 54.3 -> 84.7 mm, vias 0 -> 1
- net VDC: track 22.1 -> 50.9 mm, vias 0 -> 6
- net GND: track 18.3 -> 7.65 mm, vias 9 -> 39
- net SENSE_CURRENT: track 13.9 -> 20.8 mm, vias 1 -> 2
- net PHASE_A: track 0.00 -> 5.33 mm, vias 0 -> 1
- net SENSE_VIN: track 17.2 -> 14.8 mm
- net FET_A_L: track 22.5 -> 23.3 mm
- added copper zone on layer 1, net VDC
- added copper zone on layer 16, net VDC
- added copper zone on layer 1, net VDD_3V3
- added copper zone on layer 16, net VDD_3V3

Commit message: Currennt measurement update
Parts:
- added C16: 0.1µF, rc:C0402
- added IC6: LMV331, misc:SOT23-5L
- added R12: 3K9, rc:R0402
- added R14: DNM, rc:R0402
- added R16, R17: 000, rc:R0402
- IC5: value INA180A1 -> INA180A2
- moved C12 7.97 mm to (-12.1, 66.8), flipped to the bottom, turned to 270 degrees
- moved C14 2.64 mm to (-14.3, 69.4), turned to 0 degrees
- moved IC5 2.50 mm to (-13.4, 71.5), turned to 90 degrees
- moved R10 0.21 mm to (-3.86, 67.0)
- moved R5 0.21 mm to (-6.36, 64.5)
- moved C15 0.07 mm to (-6.61, 62.1)
- moved R6 0.07 mm to (-5.83, 61.3)
Connections:
- removed net SENSE_CURRENT: IC1.21, IC5.1
- new net CURRENT_AMP_OUT: IC1.21, IC5.1, IC6.3
- new net N$2: IC6.1, R14.2, R16.1, R17.1
- new net OVERCURRENT_FAULT: IC6.4, R12.2, R14.1
- net GND: now also C16.1, IC6.2, R17.2
- net VDD_3V3: now also C16.2, IC6.5, R12.1, R16.2
Routing:
- net SENSE_CURRENT: track 20.8 -> 0.00 mm, vias 2 -> 0
- net CURRENT_AMP_OUT: track 0.00 -> 14.8 mm, vias 0 -> 1
- net CS-: track 6.85 -> 9.40 mm
- net CS+: track 6.91 -> 7.91 mm
- net PHASE_B: track 14.3 -> 14.9 mm
- net N$30: track 18.7 -> 19.2 mm
- net N$29: track 15.5 -> 16.1 mm
- net VDD_3V3: track 120.5 -> 120.6 mm, vias 15 -> 16
- net GND: vias 39 -> 35
