File: src/power.sch (EAGLE design)
At the start: 20 parts, among them CON1 PINHEAD_2X02-0877590414, CON2 PINHEAD_2X02-0877590414, CON3 PINHEAD_2X02-0877590414, CON5 PINHEAD_2X02-0877590414, CON6 PINHEAD_2X04-SMD-2-MALE, IC1 UCC272-VDFN-HEAVY_PCB, IC2 UCC272-VDFN-HEAVY_PCB, IC3 UCC272-VDFN-HEAVY_PCB

Commit message: initial import
Parts:
- IC1, IC2, IC3: LCSC# C47661 -> (none)
Connections:
- removed net N$7: PAD4.P$1, R1.1
- new net VBAT-: CON6.6, PAD4.P$1, R1.1
- net C_PH: now also CON6.1; no longer CON6.6
- net VDC: now also CON6.8
- net VDD_15V: now also CON6.3
Other:
- moved on the sheet: CON6, PAD4, PAD5

Commit message: Updates here and there
Parts:
- added CON4, CON7: PINHEAD_2X02-0877590414, pinhead:PINHEAD_2X02-0877590414
Connections:
- net PGND: now also CON7.1, CON7.2, CON7.3, CON7.4
- net VDC: now also CON4.1, CON4.2, CON4.3, CON4.4
Changed lines of the file:
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@@
 <part name="+P9" library="supply_symbols" library_urn="urn:adsk.eagle:library:13097679" deviceset="15V" device=""/>
 <part name="+P10" library="supply_symbols" library_urn="urn:adsk.eagle:library:5017758" deviceset="VDC" device=""/>
+<part name="CON4" library="pinhead" library_urn="urn:adsk.eagle:library:2540341" deviceset="PINHEAD_2X02" device="-0877590414" package3d_urn="urn:adsk.eagle:package:23512771/2" value="PINHEAD_2X02-0877590414"/>
+<part name="+P11" library="supply_symbols" library_urn="urn:adsk.eagle:library:5017758" deviceset="VDC" device=""/>
+<part name="+P12" library="supply_symbols" library_urn="urn:adsk.eagle:library:5017758" deviceset="VDC" device=""/>
+<part name="CON7" library="pinhead" library_urn="urn:adsk.eagle:library:2540341" deviceset="PINHEAD_2X02" device="-0877590414" package3d_urn="urn:adsk.eagle:package:23512771/2" value="PINHEAD_2X02-0877590414"/>
 </parts>
 <sheets>
@@
 <instance part="+P10" gate="G$1" x="55.88" y="55.88" smashed="yes">
 <attribute name="VALUE" x="55.88" y="59.436" size="1.27" layer="96" font="vector" ratio="15" align="center"/>
+</instance>
+<instance part="CON4" gate="G$1" x="109.22" y="30.48" smashed="yes">
+<attribute name="NAME" x="115.824" y="39.37" size="1.778" layer="95" font="vector" ratio="15" align="center"/>
+</instance>
+<instance part="+P11" gate="G$1" x="104.14" y="38.1" smashed="yes">
+<attribute name="VALUE" x="104.14" y="41.656" size="1.27" layer="96" font="vector" ratio="15" align="center"/>
+</instance>
+<instance part="+P12" gate="G$1" x="127" y="38.1" smashed="yes">
+<attribute name="VALUE" x="127" y="41.656" size="1.27" layer="96" font="vector" ratio="15" align="center"/>
+</instance>
+<instance part="CON7" gate="G$1" x="154.94" y="60.96" smashed="yes">
+<attribute name="NAME" x="161.544" y="69.85" size="1.778" layer="95" font="vector" ratio="15" align="center"/>
 </instance>
 </instances>
@@
 <junction x="144.78" y="58.42"/>
 <wire x1="154.94" y1="58.42" x2="144.78" y2="58.42" width="0.1524" layer="91"/>
+<pinref part="CON7" gate="G$1" pin="1"/>
+<wire x1="152.4" y1="66.04" x2="144.78" y2="66.04" width="0.1524" layer="91"/>
+<pinref part="CON7" gate="G$1" pin="3"/>
+<wire x1="152.4" y1="63.5" x2="144.78" y2="63.5" width="0.1524" layer="91"/>
+<pinref part="CON7" gate="G$1" pin="2"/>
+<wire x1="170.18" y1="66.04" x2="172.72" y2="66.04" width="0.1524" layer="91"/>
+<wire x1="172.72" y1="66.04" x2="172.72" y2="71.12" width="0.1524" layer="91"/>
+<wire x1="172.72" y1="71.12" x2="144.78" y2="71.12" width="0.1524" layer="91"/>
+<pinref part="CON7" gate="G$1" pin="4"/>
+<wire x1="170.18" y1="63.5" x2="172.72" y2="63.5" width="0.1524" layer="91"/>
+<wire x1="172.72" y1="63.5" x2="172.72" y2="58.42" width="0.1524" layer="91"/>
+<wire x1="172.72" y1="58.42" x2="154.94" y2="58.42" width="0.1524" layer="91"/>
+<junction x="154.94" y="58.42"/>
 </segment>
 </net>
@@
 <wire x1="55.88" y1="50.8" x2="38.1" y2="50.8" width="0.1524" layer="91"/>
 </segment>
+<segment>
+<pinref part="CON4" gate="G$1" pin="1"/>
+<wire x1="106.68" y1="35.56" x2="104.14" y2="35.56" width="0.1524" layer="91"/>
+<pinref part="+P11" gate="G$1" pin="VDC"/>
+<wire x1="104.14" y1="35.56" x2="104.14" y2="38.1" width="0.1524" layer="91"/>
+<pinref part="CON4" gate="G$1" pin="3"/>
+<wire x1="106.68" y1="33.02" x2="104.14" y2="33.02" width="0.1524" layer="91"/>
+<wire x1="104.14" y1="33.02" x2="104.14" y2="35.56" width="0.1524" layer="91"/>
+<junction x="104.14" y="35.56"/>
+</segment>
+<segment>
+<pinref part="+P12" gate="G$1" pin="VDC"/>
+<pinref part="CON4" gate="G$1" pin="4"/>
+<wire x1="127" y1="38.1" x2="127" y2="35.56" width="0.1524" layer="91"/>
+<wire x1="127" y1="35.56" x2="127" y2="33.02" width="0.1524" layer="91"/>
+<wire x1="127" y1="33.02" x2="124.46" y2="33.02" width="0.1524" layer="91"/>
+<pinref part="CON4" gate="G$1" pin="2"/>
+<wire x1="124.46" y1="35.56" x2="127" y2="35.56" width="0.1524" layer="91"/>
+<junction x="127" y="35.56"/>
+</segment>
 </net>

Commit message: Currennt measurement update
Parts:
- R1: value 500 µOhms -> 200 µOhms; device SHUNT_RESISTORS:CURRENT_SHUNT_KELVIN-0.0005R-3920-KELVIN -> SHUNT_RESISTORS:CURRENT_SHUNT_KELVIN-0.0002R-3920-KELVIN; LCSC# (none) -> C469432
Changed lines of the file:
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@@
 <part name="CON2" library="pinhead" library_urn="urn:adsk.eagle:library:2540341" deviceset="PINHEAD_2X02" device="-0877590414" package3d_urn="urn:adsk.eagle:package:23512771/2" value="PINHEAD_2X02-0877590414"/>
 <part name="CON3" library="pinhead" library_urn="urn:adsk.eagle:library:2540341" deviceset="PINHEAD_2X02" device="-0877590414" package3d_urn="urn:adsk.eagle:package:23512771/2" value="PINHEAD_2X02-0877590414"/>
-<part name="R1" library="SHUNT_RESISTORS" library_urn="urn:adsk.eagle:library:2644450" deviceset="CURRENT_SHUNT_KELVIN" device="-3920-KELVIN" package3d_urn="urn:adsk.eagle:package:10874636/2" technology="-0.0005R" value="500 µOhms"/>
+<part name="R1" library="SHUNT_RESISTORS" library_urn="urn:adsk.eagle:library:2644450" deviceset="CURRENT_SHUNT_KELVIN" device="-3920-KELVIN" package3d_urn="urn:adsk.eagle:package:10874636/3" technology="-0.0002R" value="200 µOhms">
+<attribute name="LCSC#" value="C469432"/>
+</part>
 <part name="CON1" library="pinhead" library_urn="urn:adsk.eagle:library:2540341" deviceset="PINHEAD_2X02" device="-0877590414" package3d_urn="urn:adsk.eagle:package:23512771/2" value="PINHEAD_2X02-0877590414"/>
 <part name="CON5" library="pinhead" library_urn="urn:adsk.eagle:library:2540341" deviceset="PINHEAD_2X02" device="-0877590414" package3d_urn="urn:adsk.eagle:package:23512771/2" value="PINHEAD_2X02-0877590414"/>
@@
 <attribute name="NAME" x="141.986" y="40.64" size="1.778" layer="95" font="vector" ratio="15" rot="R270" align="center"/>
 <attribute name="VALUE" x="147.32" y="40.64" size="1.016" layer="95" font="vector" ratio="15" rot="R90" align="center"/>
+<attribute name="LCSC#" x="144.78" y="40.64" size="1.778" layer="96" rot="R90" display="off"/>
 </instance>
 <instance part="CON1" gate="G$1" x="109.22" y="60.96" smashed="yes">
