File: src/power.brd (EAGLE design)
At the start: 37.8 x 80 mm, 56 parts, among them CON1 PINHEAD_2X02-0877590414, CON2 PINHEAD_2X02-0877590414, CON3 PINHEAD_2X02-0877590414, CON5 PINHEAD_2X02-0877590414, CON6 PINHEAD_2X04-SMD-2-MALE, IC1 UCC272-VDFN-HEAVY_PCB, IC2 UCC272-VDFN-HEAVY_PCB, IC3 UCC272-VDFN-HEAVY_PCB, Q101 BSC077N12NS3GATMA1, Q102 BSC077N12NS3GATMA1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

Commit message: initial import
Parts:
- moved CON1 47.1 mm to (-15.7, 58.0)
- moved CON5 47.1 mm to (15.7, 58.0)
- moved PAD4 3.50 mm to (-15.5, 77.0)
- moved PAD5 3.50 mm to (15.5, 77.0)
- moved C4 0.74 mm to (4.00, 74.0), turned to 0 degrees
- moved C3 0.15 mm to (5.95, 74.0)
Connections:
- removed net N$7: PAD4.P$1, R1.1, R1.11
- new net VBAT-: CON6.6, PAD4.P$1, R1.1, R1.11
- net C_PH: now also CON6.1; no longer CON6.6
- net VDC: now also CON6.8
- net VDD_15V: now also CON6.3
Routing:
- net VDC: track 0.00 -> 19.5 mm, vias 0 -> 3
- net VDD_15V: track 43.8 -> 55.2 mm, vias 4 -> 6
- net VBAT-: track 0.00 -> 8.28 mm
- net C_PH: track 20.8 -> 17.0 mm
- net PGND: track 30.6 -> 28.0 mm
- added copper zone on layer 1, net VBAT-
- removed copper zone on layer 1, net N$7
Other:
- board size 37.8 x 80 mm -> 36 x 88.5 mm

Commit message: Updates here and there
Parts:
- added CON4, CON7: PINHEAD_2X02-0877590414, pinhead:2X02-SMD-2-MALE
- moved CON1 1.00 mm to (-15.7, 57.0)
- moved CON5 1.00 mm to (15.7, 57.0)
Connections:
- net PGND: now also CON7.1, CON7.2, CON7.3, CON7.4
- net VDC: now also CON4.1, CON4.2, CON4.3, CON4.4
Changed lines of the file:
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@@
 <setting verticaltext="up"/>
 </settings>
-<grid distance="0.2" unitdist="mm" unit="mm" style="lines" multiple="1" display="yes" altdistance="1" altunitdist="mm" altunit="mm"/>
+<grid distance="0.5" unitdist="mm" unit="mm" style="lines" multiple="1" display="yes" altdistance="1" altunitdist="mm" altunit="mm"/>
 <layers>
 <layer number="1" name="Top" color="4" fill="1" visible="yes" active="yes"/>
@@
 <attribute name="TOLERANCE" value="±1%" x="-13.8" y="68.2" size="1.778" layer="27" rot="R270" display="off"/>
 </element>
-<element name="CON1" library="pinhead" library_urn="urn:adsk.eagle:library:2540341" package="2X02-SMD-2-MALE" package3d_urn="urn:adsk.eagle:package:23512771/2" value="PINHEAD_2X02-0877590414" x="-15.7" y="58" smashed="yes" rot="R90">
-<attribute name="DIGIKEY#" value="WM18712-ND" x="-15.7" y="58" size="1.778" layer="27" rot="R90" display="off"/>
-<attribute name="MANF" value="Molex" x="-15.7" y="58" size="1.778" layer="27" rot="R90" display="off"/>
-<attribute name="MANF#" value="0877590414" x="-15.7" y="58" size="1.778" layer="27" rot="R90" display="off"/>
-<attribute name="NAME" x="-15.7" y="58" size="1.27" layer="25" font="vector" ratio="15" align="center"/>
-</element>
-<element name="CON5" library="pinhead" library_urn="urn:adsk.eagle:library:2540341" package="2X02-SMD-2-MALE" package3d_urn="urn:adsk.eagle:package:23512771/2" value="PINHEAD_2X02-0877590414" x="15.7" y="58" smashed="yes" rot="R90">
-<attribute name="DIGIKEY#" value="WM18712-ND" x="15.7" y="58" size="1.778" layer="27" rot="R90" display="off"/>
-<attribute name="MANF" value="Molex" x="15.7" y="58" size="1.778" layer="27" rot="R90" display="off"/>
-<attribute name="MANF#" value="0877590414" x="15.7" y="58" size="1.778" layer="27" rot="R90" display="off"/>
-<attribute name="NAME" x="15.7" y="58" size="1.27" layer="25" font="vector" ratio="15" align="center"/>
+<element name="CON1" library="pinhead" library_urn="urn:adsk.eagle:library:2540341" package="2X02-SMD-2-MALE" package3d_urn="urn:adsk.eagle:package:23512771/2" value="PINHEAD_2X02-0877590414" x="-15.7" y="57" smashed="yes" rot="R90">
+<attribute name="DIGIKEY#" value="WM18712-ND" x="-15.7" y="57" size="1.778" layer="27" rot="R90" display="off"/>
+<attribute name="MANF" value="Molex" x="-15.7" y="57" size="1.778" layer="27" rot="R90" display="off"/>
+<attribute name="MANF#" value="0877590414" x="-15.7" y="57" size="1.778" layer="27" rot="R90" display="off"/>
+<attribute name="NAME" x="-15.7" y="57" size="1.27" layer="25" font="vector" ratio="15" align="center"/>
+</element>
+<element name="CON5" library="pinhead" library_urn="urn:adsk.eagle:library:2540341" package="2X02-SMD-2-MALE" package3d_urn="urn:adsk.eagle:package:23512771/2" value="PINHEAD_2X02-0877590414" x="15.7" y="57" smashed="yes" rot="R90">
+<attribute name="DIGIKEY#" value="WM18712-ND" x="15.7" y="57" size="1.778" layer="27" rot="R90" display="off"/>
+<attribute name="MANF" value="Molex" x="15.7" y="57" size="1.778" layer="27" rot="R90" display="off"/>
+<attribute name="MANF#" value="0877590414" x="15.7" y="57" size="1.778" layer="27" rot="R90" display="off"/>
+<attribute name="NAME" x="15.7" y="57" size="1.27" layer="25" font="vector" ratio="15" align="center"/>
 </element>
 <element name="CON6" library="pinhead" library_urn="urn:adsk.eagle:library:2540341" package="2X04-SMD-2-MALE" package3d_urn="urn:adsk.eagle:package:23791919/2" value="PINHEAD_2X04-SMD-2-MALE" x="-5.15" y="75.4" smashed="yes" rot="R180">
@@
 <attribute name="MANF#" value="0877590814" x="-5.15" y="75.4" size="1.778" layer="27" rot="R180" display="off"/>
 <attribute name="NAME" x="-5.15" y="75.4" size="1.27" layer="25" font="vector" ratio="15" rot="R90" align="center"/>
+</element>
+<element name="CON4" library="pinhead" library_urn="urn:adsk.eagle:library:2540341" package="2X02-SMD-2-MALE" package3d_urn="urn:adsk.eagle:package:23512771/2" value="PINHEAD_2X02-0877590414" x="15.7" y="13" smashed="yes" rot="R90">
+<attribute name="DIGIKEY#" value="WM18712-ND" x="16.2" y="13" size="1.778" layer="27" rot="R90" display="off"/>
+<attribute name="MANF" value="Molex" x="16.2" y="13" size="1.778" layer="27" rot="R90" display="off"/>
+<attribute name="MANF#" value="0877590414" x="16.2" y="13" size="1.778" layer="27" rot="R90" display="off"/>
+<attribute name="NAME" x="15.7" y="13" size="1.27" layer="25" font="vector" ratio="15" align="center"/>
+</element>
+<element name="CON7" library="pinhead" library_urn="urn:adsk.eagle:library:2540341" package="2X02-SMD-2-MALE" package3d_urn="urn:adsk.eagle:package:23512771/2" value="PINHEAD_2X02-0877590414" x="-15.7" y="13" smashed="yes" rot="R90">
+<attribute name="DIGIKEY#" value="WM18712-ND" x="-15.7" y="13" size="1.778" layer="27" rot="R90" display="off"/>
+<attribute name="MANF" value="Molex" x="-15.7" y="13" size="1.778" layer="27" rot="R90" display="off"/>
+<attribute name="MANF#" value="0877590414" x="-15.7" y="13" size="1.778" layer="27" rot="R90" display="off"/>
+<attribute name="NAME" x="-15.7" y="13" size="1.27" layer="25" font="vector" ratio="15" align="center"/>
 </element>
 </elements>
@@
 <wire x1="0.89853125" y1="23" x2="1.1" y2="23" width="0.4" layer="1"/>
 <wire x1="0.775" y1="19.9" x2="0.7" y2="22.6" width="0.4" layer="1"/>
-<via x="-15.55" y="15.8" extent="1-16" drill="0.4" diameter="0.7"/>
+<via x="-15.55" y="19.8" extent="1-16" drill="0.4" diameter="0.7"/>
 <polygon width="0.4" layer="16">
 <vertex x="-0.9" y="78.55"/>
@@
 <wire x1="-4.5" y1="75.1" x2="-9.45" y2="70.15" width="1" layer="16"/>
 <wire x1="4.725" y1="74" x2="4.725" y2="75" width="0.4" layer="1"/>
+<contactref element="CON7" pad="1"/>
+<contactref element="CON7" pad="3"/>
+<contactref element="CON7" pad="2"/>
+<contactref element="CON7" pad="4"/>
 </signal>
 <signal name="VDC" class="1">
@@
 <vertex x="-4.75" y="78.05"/>
 </polygon>
+<contactref element="CON4" pad="1"/>
+<contactref element="CON4" pad="3"/>
+<contactref element="CON4" pad="4"/>
+<contactref element="CON4" pad="2"/>
 </signal>
 <signal name="PHASE_A:N$3" class="1">

Commit message: Currennt measurement update
Parts:
- R1: value 500 µOhms -> 200 µOhms
Changed lines of the file:
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@@
 <attribute name="NAME" x="-5.25" y="24.4" size="1.27" layer="25" font="vector" ratio="15" rot="R90" align="center"/>
 </element>
-<element name="R1" library="SHUNT_RESISTORS" library_urn="urn:adsk.eagle:library:2644450" package="R3920-KELVIN" package3d_urn="urn:adsk.eagle:package:10874636/2" value="500 µOhms" x="-13.8" y="68.2" smashed="yes" rot="R270">
-<attribute name="DIGIKEY#" value="CSS2H-3920R-L500FCT-ND" x="-13.8" y="68.2" size="1.778" layer="27" rot="R270" display="off"/>
+<element name="R1" library="SHUNT_RESISTORS" library_urn="urn:adsk.eagle:library:2644450" package="R3920-KELVIN" package3d_urn="urn:adsk.eagle:package:10874636/3" value="200 µOhms" x="-13.8" y="68.2" smashed="yes" rot="R270">
+<attribute name="DIGIKEY#" value="CSS2H-3920R-L200FCT-ND" x="-13.8" y="68.2" size="1.778" layer="27" rot="R270" display="off"/>
+<attribute name="LCSC#" value="C469432" x="-13.8" y="68.2" size="1.778" layer="27" rot="R270" display="off"/>
 <attribute name="MANF" value="Bourns Inc" x="-13.8" y="68.2" size="1.778" layer="27" rot="R270" display="off"/>
-<attribute name="MANF#" value="CSS2H-3920R-L500F" x="-13.8" y="68.2" size="1.778" layer="27" rot="R270" display="off"/>
+<attribute name="MANF#" value="CSS2H-3920R-L200FCT-ND" x="-13.8" y="68.2" size="1.778" layer="27" rot="R270" display="off"/>
 <attribute name="NAME" x="-13.8" y="68.2" size="1.5" layer="25" font="vector" ratio="15" rot="R270" align="center"/>
 <attribute name="OPERATING_TEMP" value="-55°C ~ 170°C" x="-13.8" y="68.2" size="1.778" layer="27" rot="R270" display="off"/>
 <attribute name="PACKAGE" value="3920" x="-13.8" y="68.2" size="1.778" layer="27" rot="R270" display="off"/>
-<attribute name="POWER" value="9W" x="-13.8" y="68.2" size="1.778" layer="27" rot="R270" display="off"/>
+<attribute name="POWER" value="12W" x="-13.8" y="68.2" size="1.778" layer="27" rot="R270" display="off"/>
 <attribute name="TC" value="±50ppm/°C" x="-13.8" y="68.2" size="1.778" layer="27" rot="R270" display="off"/>
 <attribute name="TOLERANCE" value="±1%" x="-13.8" y="68.2" size="1.778" layer="27" rot="R270" display="off"/>
