File: src/connectors.brd (EAGLE design)
At the start: 36 x 14.4 mm, 11 parts, among them CON1 CON-4P-TABS-JST_GH-RA, CON2 CON-4P-TABS-JST_GH-RA, CON3 PINHEAD_1X04-2, CON4 PINHEAD_1X04-2, IC6 TJA1051-HVSON8, IC8 TPD3S014DBVR-SOT23-6

Commit message: Connectors PCB UAVCAN logo added
Parts:
- added U$1: (no value), logo:UAVCAN_10X3
Changed lines of the file:
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@@
 <setting verticaltext="up"/>
 </settings>
-<grid distance="0.05" unitdist="mm" unit="mm" style="lines" multiple="1" display="yes" altdistance="5" altunitdist="mil" altunit="mil"/>
+<grid distance="0.5" unitdist="mm" unit="mm" style="lines" multiple="10" display="yes" altdistance="5" altunitdist="mil" altunit="mil"/>
 <layers>
-<layer number="1" name="Top" color="4" fill="1" visible="yes" active="yes"/>
+<layer number="1" name="Top" color="4" fill="1" visible="no" active="yes"/>
 <layer number="2" name="Route2" color="16" fill="1" visible="no" active="no"/>
 <layer number="3" name="Route3" color="17" fill="1" visible="no" active="no"/>
@@
 <layer number="14" name="Route14" color="22" fill="1" visible="no" active="no"/>
 <layer number="15" name="Route15" color="23" fill="1" visible="no" active="no"/>
-<layer number="16" name="Bottom" color="1" fill="1" visible="no" active="yes"/>
+<layer number="16" name="Bottom" color="1" fill="1" visible="yes" active="yes"/>
 <layer number="17" name="Pads" color="2" fill="1" visible="yes" active="yes"/>
 <layer number="18" name="Vias" color="2" fill="1" visible="yes" active="yes"/>
 <layer number="19" name="Unrouted" color="6" fill="1" visible="yes" active="yes"/>
 <layer number="20" name="Dimension" color="24" fill="1" visible="yes" active="yes"/>
-<layer number="21" name="tPlace" color="7" fill="1" visible="yes" active="yes"/>
+<layer number="21" name="tPlace" color="7" fill="1" visible="no" active="yes"/>
 <layer number="22" name="bPlace" color="7" fill="1" visible="yes" active="yes"/>
-<layer number="23" name="tOrigins" color="15" fill="1" visible="yes" active="yes"/>
+<layer number="23" name="tOrigins" color="15" fill="1" visible="no" active="yes"/>
 <layer number="24" name="bOrigins" color="15" fill="1" visible="yes" active="yes"/>
-<layer number="25" name="tNames" color="7" fill="1" visible="yes" active="yes"/>
+<layer number="25" name="tNames" color="7" fill="1" visible="no" active="yes"/>
 <layer number="26" name="bNames" color="7" fill="1" visible="yes" active="yes"/>
 <layer number="27" name="tValues" color="7" fill="1" visible="no" active="yes"/>
@@
 <layer number="49" name="Reference" color="7" fill="1" visible="no" active="yes"/>
 <layer number="50" name="dxf" color="7" fill="1" visible="no" active="no"/>
-<layer number="51" name="tDocu" color="7" fill="1" visible="yes" active="yes"/>
+<layer number="51" name="tDocu" color="7" fill="1" visible="no" active="yes"/>
 <layer number="52" name="bDocu" color="7" fill="1" visible="yes" active="yes"/>
 <layer number="53" name="tGND_GNDA" color="7" fill="9" visible="no" active="no"/>
@@
 <attribute name="NAME" x="-18.4" y="69.8" size="1" layer="25" font="vector" ratio="15" rot="R90" align="center"/>
 </element>
+<element name="U$1" library="logo" library_urn="urn:adsk.eagle:library:6668987" package="UAVCAN_10X3" package3d_urn="urn:adsk.eagle:package:11612836/1" value="" x="5.1" y="75.7" smashed="yes" rot="MR0"/>
 </elements>
 <signals>

Commit message: Silkscreen updates
Parts:
- moved U$1 1.50 mm to (5.10, 77.2)
Other:
- board text added: "Valenok connectors PCB V0.1"
Changed lines of the file:
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@@
 <setting verticaltext="up"/>
 </settings>
-<grid distance="0.5" unitdist="mm" unit="mm" style="lines" multiple="10" display="yes" altdistance="5" altunitdist="mil" altunit="mil"/>
+<grid distance="0.1" unitdist="mm" unit="mm" style="lines" multiple="10" display="yes" altdistance="5" altunitdist="mil" altunit="mil"/>
 <layers>
 <layer number="1" name="Top" color="4" fill="1" visible="no" active="yes"/>
@@
 </layers>
 <board>
-<fusionsync huburn="a.cGVyc29uYWw6dWUyYWE4ZDY4" projecturn="a.cGVyc29uYWw6dWUyYWE4ZDY4IzIwMjAwOTI1MzM2NDYxMjgx" f3durn="urn:adsk.wipprod:dm.lineage:5f-RR5beSAqgs6k1iF_brA" pcbguid="" lastpulledtime="" lastsyncedchangeguid="" latestrevisionid="04173ad2-e432-4cf5-9b9d-9b2dc3d49b22" lastsyncedrevisionid="04173ad2-e432-4cf5-9b9d-9b2dc3d49b22" lastboardhashguid="f24dbab6-befe-c805-d208-4619c0b274fc" lastpushedtime="2020-11-10T14:33:02Z" linktopcb3d="true"/>
+<fusionsync huburn="a.cGVyc29uYWw6dWUyYWE4ZDY4" projecturn="a.cGVyc29uYWw6dWUyYWE4ZDY4IzIwMjAwOTI1MzM2NDYxMjgx" f3durn="urn:adsk.wipprod:dm.lineage:5f-RR5beSAqgs6k1iF_brA" pcbguid="" lastpulledtime="" lastsyncedchangeguid="" latestrevisionid="c05a1ed8-b5ef-45bf-99de-9ff0bf12f278" lastsyncedrevisionid="c05a1ed8-b5ef-45bf-99de-9ff0bf12f278" lastboardhashguid="171d5d68-3516-144f-ad2e-87fcf70b681d" lastpushedtime="2020-11-16T10:40:15Z" linktopcb3d="true"/>
 <plain>
 <wire x1="5.5" y1="75.1" x2="5.5" y2="74.1" width="0.1524" layer="138"/>
@@
 <wire x1="16.6" y1="69.8" x2="17" y2="69.8" width="0.01" layer="138"/>
 <wire x1="16.8" y1="70" x2="16.8" y2="69.6" width="0.01" layer="138"/>
+<text x="-11" y="76.9" size="1.4" layer="22" font="vector" ratio="15" rot="MR0" align="center">Valenok
+connectors
+PCB V0.1</text>
 </plain>
 <attributes>
@@
 <attribute name="NAME" x="-18.4" y="69.8" size="1" layer="25" font="vector" ratio="15" rot="R90" align="center"/>
 </element>
-<element name="U$1" library="logo" library_urn="urn:adsk.eagle:library:6668987" package="UAVCAN_10X3" package3d_urn="urn:adsk.eagle:package:11612836/1" value="" x="5.1" y="75.7" smashed="yes" rot="MR0"/>
+<element name="U$1" library="logo" library_urn="urn:adsk.eagle:library:6668987" package="UAVCAN_10X3" package3d_urn="urn:adsk.eagle:package:11612836/1" value="" x="5.1" y="77.2" smashed="yes" rot="MR0"/>
 </elements>
 <signals>
@@
 </drawing>
 <compatibility>
+<note version="6.3" minversion="6.2.2" severity="warning">
+Since Version 6.2.2 text objects can contain more than one line,
+which will not be processed correctly with this version.
+</note>
 <note version="8.2" severity="warning">
 Since Version 8.2, EAGLE supports online libraries. The ids

Commit message: assembly variant update
Parts:
- flipped CON3 to the bottom
- flipped CON4 to the bottom
Changed lines of the file:
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@@
 <grid distance="0.1" unitdist="mm" unit="mm" style="lines" multiple="10" display="yes" altdistance="5" altunitdist="mil" altunit="mil"/>
 <layers>
-<layer number="1" name="Top" color="4" fill="1" visible="no" active="yes"/>
+<layer number="1" name="Top" color="4" fill="1" visible="yes" active="yes"/>
 <layer number="2" name="Route2" color="16" fill="1" visible="no" active="no"/>
 <layer number="3" name="Route3" color="17" fill="1" visible="no" active="no"/>
@@
 <layer number="19" name="Unrouted" color="6" fill="1" visible="yes" active="yes"/>
 <layer number="20" name="Dimension" color="24" fill="1" visible="yes" active="yes"/>
-<layer number="21" name="tPlace" color="7" fill="1" visible="no" active="yes"/>
+<layer number="21" name="tPlace" color="7" fill="1" visible="yes" active="yes"/>
 <layer number="22" name="bPlace" color="7" fill="1" visible="yes" active="yes"/>
-<layer number="23" name="tOrigins" color="15" fill="1" visible="no" active="yes"/>
+<layer number="23" name="tOrigins" color="15" fill="1" visible="yes" active="yes"/>
 <layer number="24" name="bOrigins" color="15" fill="1" visible="yes" active="yes"/>
-<layer number="25" name="tNames" color="7" fill="1" visible="no" active="yes"/>
+<layer number="25" name="tNames" color="7" fill="1" visible="yes" active="yes"/>
 <layer number="26" name="bNames" color="7" fill="1" visible="yes" active="yes"/>
 <layer number="27" name="tValues" color="7" fill="1" visible="no" active="yes"/>
@@
 <layer number="49" name="Reference" color="7" fill="1" visible="no" active="yes"/>
 <layer number="50" name="dxf" color="7" fill="1" visible="no" active="no"/>
-<layer number="51" name="tDocu" color="7" fill="1" visible="no" active="yes"/>
+<layer number="51" name="tDocu" color="7" fill="1" visible="yes" active="yes"/>
 <layer number="52" name="bDocu" color="7" fill="1" visible="yes" active="yes"/>
 <layer number="53" name="tGND_GNDA" color="7" fill="9" visible="no" active="no"/>
@@
 </attributes>
 <variantdefs>
-<variantdef name="basic"/>
+<variantdef name="basic" current="yes"/>
 </variantdefs>
 <classes>
@@
 <attribute name="VOLTAGE" value="6.3V" x="12" y="84.1" size="1.778" layer="27" rot="R180" display="off"/>
 </element>
-<element name="CON3" library="pinhead" library_urn="urn:adsk.eagle:library:2540341" package="1X04-PTH-2" package3d_urn="urn:adsk.eagle:package:4854340/4" value="PINHEAD_1X04-2" x="16.8" y="69.8" smashed="yes" rot="R270">
-<attribute name="NAME" x="18.4" y="69.8" size="1" layer="25" font="vector" ratio="15" rot="R270" align="center"/>
-</element>
-<element name="CON4" library="pinhead" library_urn="urn:adsk.eagle:library:2540341" package="1X04-PTH-2" package3d_urn="urn:adsk.eagle:package:4854340/4" value="PINHEAD_1X04-2" x="-16.8" y="69.8" smashed="yes" rot="R90">
-<attribute name="NAME" x="-18.4" y="69.8" size="1" layer="25" font="vector" ratio="15" rot="R90" align="center"/>
+<element name="CON3" library="pinhead" library_urn="urn:adsk.eagle:library:2540341" package="1X04-PTH-2" package3d_urn="urn:adsk.eagle:package:4854340/4" value="PINHEAD_1X04-2" x="16.8" y="69.8" populate="no" smashed="yes" rot="MR270">
+<attribute name="NAME" x="15.2" y="69.8" size="1" layer="26" font="vector" ratio="15" rot="MR270" align="center"/>
+</element>
+<element name="CON4" library="pinhead" library_urn="urn:adsk.eagle:library:2540341" package="1X04-PTH-2" package3d_urn="urn:adsk.eagle:package:4854340/4" value="PINHEAD_1X04-2" x="-16.8" y="69.8" populate="no" smashed="yes" rot="MR90">
+<attribute name="NAME" x="-15.2" y="69.8" size="1" layer="26" font="vector" ratio="15" rot="MR90" align="center"/>
 </element>
 <element name="U$1" library="logo" library_urn="urn:adsk.eagle:library:6668987" package="UAVCAN_10X3" package3d_urn="urn:adsk.eagle:package:11612836/1" value="" x="5.1" y="77.2" smashed="yes" rot="MR0"/>

Commit message: Outline updates to allow debug assembly with connectors
Parts:
- CON3, CON4: value PINHEAD_1X04-2 -> PINHEAD_1X04-2-FEMALE; device pinhead:1X04-PTH-2 -> pinhead:1X04-PTH-2-FEMALE
Changed lines of the file:
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@@
 </attributes>
 <variantdefs>
-<variantdef name="basic" current="yes"/>
+<variantdef name="basic"/>
 </variantdefs>
 <classes>
@@
 <attribute name="VOLTAGE" value="6.3V" x="12" y="84.1" size="1.778" layer="27" rot="R180" display="off"/>
 </element>
-<element name="CON3" library="pinhead" library_urn="urn:adsk.eagle:library:2540341" package="1X04-PTH-2" package3d_urn="urn:adsk.eagle:package:4854340/4" value="PINHEAD_1X04-2" x="16.8" y="69.8" populate="no" smashed="yes" rot="MR270">
+<element name="CON3" library="pinhead" library_urn="urn:adsk.eagle:library:2540341" package="1X04-PTH-2-FEMALE" package3d_urn="urn:adsk.eagle:package:6503396/2" value="PINHEAD_1X04-2-FEMALE" x="16.8" y="69.8" smashed="yes" rot="MR270">
 <attribute name="NAME" x="15.2" y="69.8" size="1" layer="26" font="vector" ratio="15" rot="MR270" align="center"/>
 </element>
-<element name="CON4" library="pinhead" library_urn="urn:adsk.eagle:library:2540341" package="1X04-PTH-2" package3d_urn="urn:adsk.eagle:package:4854340/4" value="PINHEAD_1X04-2" x="-16.8" y="69.8" populate="no" smashed="yes" rot="MR90">
+<element name="CON4" library="pinhead" library_urn="urn:adsk.eagle:library:2540341" package="1X04-PTH-2-FEMALE" package3d_urn="urn:adsk.eagle:package:6503396/2" value="PINHEAD_1X04-2-FEMALE" x="-16.8" y="69.8" smashed="yes" rot="MR90">
 <attribute name="NAME" x="-15.2" y="69.8" size="1" layer="26" font="vector" ratio="15" rot="MR90" align="center"/>
 </element>
