File: src/A/logic.brd (EAGLE design)
At the start: 36 x 73.5 mm, 89 parts, among them CON1 CON-4P-TABS-JST_GH-RA, CON11 PINHEAD_1X04-2, CON12 PINHEAD_1X04-2, CON2 PINHEAD_1X04-2.54, CON3 PINHEAD_2X04-PLS-2, CON6 PINHEAD_2X02-PTH-2-MALE, CON7 PINHEAD_2X02-PTH-2-MALE, IC1 STM32F105RCT6, IC10 LM75-TSSOP8, IC101 LM5017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

Commit message: variant A updates
Parts:
- R1: value 000 -> DNM
Connections:
- net VDD_3V3: no longer CON11.1
- net VDD_5V: now also CON11.1
Routing:
- net VDD_5V: track 11.2 -> 50.8 mm
- net VDD_3V3: track 208.6 -> 201.2 mm, vias 21 -> 22
- net GND: vias 83 -> 81
- added copper zone on layer 15, net VDD_5V
